File: Hardware/C10W1B1V1.0/Kicad/C10W1B1V1.0.kicad_pcb (KiCad board)
At the start: 2 copper layers, 25 parts, among them IC1 STM32L412K8U6, IC2 TSC101AILT, Q1 STL300N4LF8, Q2 SI7155DP-T1-GE3, Q3 STL300N4LF8, Q4 SI7155DP-T1-GE3, Q5 SQ2362CES-T1_GE3, Q6 SQ2362CES-T1_GE3

Commit message: Dodano zabezpieczenia
Parts:
- removed IC1: STM32L412K8U6, Footprints:QFN50P500X500X60-33N-D
- removed IC2: TSC101AILT, Footprints:SOT95P280X145-5N
- added C1: 100n/50V/X5R, Capacitor_SMD:C_0402_1005Metric, F.Cu at (194.4, 79.1)
- added C10: 100n/50V/X5R, Capacitor_SMD:C_0402_1005Metric, F.Cu at (186.1, 89.9)
- added C11: 100n/50V/X5R, Capacitor_SMD:C_0402_1005Metric, F.Cu at (175.4, 97.8)
- added C12: 100n/50V/X5R, Capacitor_SMD:C_0402_1005Metric, F.Cu at (193.4, 81.1)
- added C13: 100n/50V/X5R, Capacitor_SMD:C_0402_1005Metric, F.Cu at (186.1, 87.9)
- added C14: 100n/50V/X5R, Capacitor_SMD:C_0402_1005Metric, F.Cu at (200.8, 72.5)
- added C15: 100n/50V/X5R, Capacitor_SMD:C_0402_1005Metric, F.Cu at (204.3, 69.7)
- added C16: 100n/50V/X5R, Capacitor_SMD:C_0402_1005Metric, F.Cu at (175.4, 99.8)
- added C17: 10u/50V/X5R, Capacitor_SMD:C_1206_3216Metric, F.Cu at (162.6, 78.9)
- added C18: 10u/10V/X5R, Capacitor_SMD:C_0805_2012Metric, F.Cu at (171.8, 98.3)
- added C19: 10u/10V/X5R, Capacitor_SMD:C_0805_2012Metric, F.Cu at (171.8, 101.3)
- added C2: RGA101M1HBK-0811G, Capacitor_THT:CP_Radial_D8.0mm_P3.50mm, F.Cu at (172.7, 72.4)
- added C20: 10u/10V/X5R, Capacitor_SMD:C_0805_2012Metric, F.Cu at (174.9, 95.3)
- added C21: 10u/10V/X5R, Capacitor_SMD:C_0805_2012Metric, F.Cu at (178.5, 90.7)
- added C22: 100n/50V/X5R, Capacitor_SMD:C_0402_1005Metric, F.Cu at (178.6, 93.2)
- added C23: 1u/50V/X5R, Capacitor_SMD:C_0402_1005Metric, F.Cu at (181.4, 93.2)
- added C24: 100p/50V/X5R, Capacitor_SMD:C_0402_1005Metric, F.Cu at (178.6, 95.2)
- added C25: 2u2/50V/X5R, Capacitor_SMD:C_0402_1005Metric, F.Cu at (197.3, 77.1)
- added C26: 10u/10V/X5R, Capacitor_SMD:C_0805_2012Metric, F.Cu at (191.2, 73.8)
- added C27: 10u/10V/X5R, Capacitor_SMD:C_0805_2012Metric, F.Cu at (178.7, 86.3)
- added C28: 1u/50V/X5R, Capacitor_SMD:C_0402_1005Metric, F.Cu at (190.5, 83.3)
- added C29: 2u2/50V/X5R, Capacitor_SMD:C_0402_1005Metric, F.Cu at (178.6, 97.2)
- added C3: 10n/50V/X5R, Capacitor_SMD:C_0402_1005Metric, F.Cu at (190.5, 85.3)
- added C30: 10u/10V/X5R, Capacitor_SMD:C_0805_2012Metric, F.Cu at (170.4, 95.3)
- added C31: 4u7/50V/X5R, Capacitor_SMD:C_0402_1005Metric, F.Cu at (124.8, 113.8)
- added C32: 4u7/50V/X5R, Capacitor_SMD:C_0402_1005Metric, F.Cu at (127.7, 111.8)
- added C33: 4u7/50V/X5R, Capacitor_SMD:C_0402_1005Metric, F.Cu at (130.6, 109.8)
- added C34: 4u7/50V/X5R, Capacitor_SMD:C_0402_1005Metric, F.Cu at (127.7, 113.8)
- added C35: 4u7/50V/X5R, Capacitor_SMD:C_0402_1005Metric, F.Cu at (130.6, 111.8)
- added C4: 10n/50V/X5R, Capacitor_SMD:C_0402_1005Metric, F.Cu at (204.3, 71.7)
- added C5: RGA101M1HBK-0811G, Capacitor_THT:CP_Radial_D8.0mm_P3.50mm, F.Cu at (145.4, 98.5)
- added C6: RGA101M1HBK-0811G, Capacitor_THT:CP_Radial_D8.0mm_P3.50mm, F.Cu at (197.4, 61.9)
- added C7: RGA101M1HBK-0811G, Capacitor_THT:CP_Radial_D8.0mm_P3.50mm, F.Cu at (135.6, 98.5)
- added C8: RGA101M1HBK-0811G, Capacitor_THT:CP_Radial_D8.0mm_P3.50mm, F.Cu at (163.0, 72.4)
- added C9: RGA101M1HBK-0811G, Capacitor_THT:CP_Radial_D8.0mm_P3.50mm, F.Cu at (125.9, 98.5)
- added D5: D_TVS, Diode_SMD:D_SMB, F.Cu at (197.7, 88.1)
- added D6: BAT54S, Package_TO_SOT_SMD:SOT-23, F.Cu at (160.4, 30.8)
- added D7: BAT54S, Package_TO_SOT_SMD:SOT-23, F.Cu at (164.9, 30.8)
- added D8: BAT54S, Package_TO_SOT_SMD:SOT-23, F.Cu at (169.3, 30.8)
- added F1: SF-1206S1500W-2, Fuse:Fuse_1206_3216Metric, F.Cu at (168.4, 86.9)
- added L1: CBC3225T100KR, Inductor_SMD:L_1210_3225Metric, F.Cu at (182.0, 77.8)
- added Q10: SQ2362CES-T1_GE3, Package_TO_SOT_SMD:SOT-23, F.Cu at (186.9, 82.6)
- added Q11: SI7155DP-T1-GE3, Footprints:SI7155DPT1GE3, F.Cu at (184.1, 71.7)
- added Q7: STL300N4LF8, Footprints:STL60N10F7, F.Cu at (155.9, 98.6)
- added Q8: SI7155DP-T1-GE3, Footprints:SI7155DPT1GE3, F.Cu at (170.5, 81.2)
- added Q9: SQ2362CES-T1_GE3, Package_TO_SOT_SMD:SOT-23, F.Cu at (167.3, 101.3)
- added R13: 10m/1%/0.063W, Resistor_SMD:R_0612_1632Metric, F.Cu at (182.6, 82.3)
- added R14: 12K/1%/0.063W, Resistor_SMD:R_0402_1005Metric, F.Cu at (182.2, 90.0)
- added R15: 22K/1%/0.063W, Resistor_SMD:R_0402_1005Metric, F.Cu at (194.5, 77.1)
- added R16: 50m/1%/0.063W, Resistor_SMD:R_2512_6332Metric, F.Cu at (198.5, 69.1)
- added R17: 12K/1%/0.063W, Resistor_SMD:R_0402_1005Metric, F.Cu at (161.2, 81.6)
- added R18: 22K/1%/0.063W, Resistor_SMD:R_0402_1005Metric, F.Cu at (191.6, 78.3)
- added R19: 10/1%/5W, Resistor_THT:R_Axial_Power_L25.0mm_W9.0mm_P30.48mm, F.Cu at (161.7, 62.4)
- added R20: 10/1%/5W, Resistor_THT:R_Axial_Power_L25.0mm_W9.0mm_P30.48mm, F.Cu at (192.2, 52.8)
- added R21: 100K/1%/0.063W, Resistor_SMD:R_0402_1005Metric, F.Cu at (191.6, 76.3)
- added R22: 10K/1%/0.063W, Resistor_SMD:R_0402_1005Metric, F.Cu at (186.1, 85.9)
- added R23: 3K3/1%/0.063W, Resistor_SMD:R_0402_1005Metric, F.Cu at (190.6, 81.3)
- added R24: 10K/1%/0.063W, Resistor_SMD:R_0402_1005Metric, F.Cu at (164.1, 81.6)
- added R25: 10K/1%/0.063W, Resistor_SMD:R_0402_1005Metric, F.Cu at (204.3, 67.7)
- added R26: 58.87K/1%/0.063W, Resistor_SMD:R_0402_1005Metric, F.Cu at (176.8, 78.2)
- added R27: 10K/1%/0.063W, Resistor_SMD:R_0402_1005Metric, F.Cu at (121.9, 109.8)
- added R28: 10K/1%/0.063W, Resistor_SMD:R_0402_1005Metric, F.Cu at (121.9, 111.8)
- added R29: 174K/1%/0.063W, Resistor_SMD:R_0402_1005Metric, F.Cu at (124.8, 109.8)
- added R30: 330K/1%/0.063W, Resistor_SMD:R_0402_1005Metric, F.Cu at (121.9, 113.8)
- added R31: 174K/1%/0.063W, Resistor_SMD:R_0402_1005Metric, F.Cu at (124.8, 111.8)
- added R32: 330K/1%/0.063W, Resistor_SMD:R_0402_1005Metric, F.Cu at (127.7, 109.8)
- added R33: 100K/1%/0.063W, Resistor_SMD:R_0402_1005Metric, F.Cu at (159.7, 34.0)
- added R34: 10K/1%/0.063W, Resistor_SMD:R_0402_1005Metric, F.Cu at (162.6, 34.0)
- added TP1: DC/DC, TestPoint:TestPoint_Pad_2.0x2.0mm, F.Cu at (177.3, 104.7)
- added U1: TSC101AILT, Footprints:SOT95P280X145-5N, F.Cu at (191.6, 70.0)
- added U10: 74HC08D,653, Footprints:SOIC127P600X175-14N, F.Cu at (161.4, 88.4)
- added U11: STM32L431CCUx, Package_DFN_QFN:QFN-48-1EP_7x7mm_P0.5mm_EP5.6x5.6mm, F.Cu at (138.7, 110.6)
- added U2: MAX16171ATA_VY+, Footprints:SON50P300X200X80-9N, F.Cu at (173.9, 87.4)
- added U3: MCP1501T-20E/CHY, Footprints:SOT95P280X145-6N, F.Cu at (162.5, 101.3)
- added U4: AP331AWG-7, Footprints:SOT95P285X145-5N, F.Cu at (168.3, 90.8)
- added U5: TSC101AILT, Footprints:SOT95P280X145-5N, F.Cu at (173.6, 91.5)
- added U6: NC7SZ74L8X, Footprints:NC7SZ74L8X, F.Cu at (182.8, 86.7)
- added U7: AP64060QWU-7, Footprints:SOT95P280X100-6N, F.Cu at (196.8, 73.8)
- added U8: AP2210K-5.0TRG1, Footprints:SOT95P282X145-5N, F.Cu at (187.5, 78.0)
- added U9: TLV74333PDBVR, Footprints:SOT95P280X145-5N, F.Cu at (178.0, 82.2)
- FL1: value 7448680140 -> SC-15-02J; footprint Footprints:7448680140 -> Footprints:SC1502J
- R1, R12, R8, R9: value 10K/1%/0.063W -> 1K/1%/0.063W
- moved R7 136.2 mm to (246.9, 58.1)
- moved Q6 135.1 mm to (243.2, 59.4)
- moved Q5 125.7 mm to (244.4, 63.9), turned to 0 degrees
- moved R1 125.1 mm to (232.7, 66.1)
- moved Q2 117.9 mm to (236.1, 61.1)
- moved R12 112.2 mm to (246.9, 60.1)
- moved R4 106.1 mm to (220.8, 78.2)
- moved R8 105.9 mm to (226.6, 77.9)
- moved Q4 104.0 mm to (221.3, 71.2)
- moved Q1 103.5 mm to (238.2, 70.0)
- moved R2 103.4 mm to (220.8, 76.2)
- moved R9 103.3 mm to (235.6, 75.8)
- moved R5 102.4 mm to (223.7, 77.9)
- moved R3 100.9 mm to (217.9, 78.2)
- moved R11 100.2 mm to (232.5, 77.9)
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Connections:
- FL1 pad 2: Net-(FL1-Pad2) -> VCC
- FL1 pad 3: Net-(FL1-Pad3) -> GND
- FL1 pad 4: Net-(FL1-Pad4) -> GND1
