File: Hardware/C10W1B1V1.0/Kicad/C10W1B1V1.0.sch (KiCad schematic (older format))
At the start: 0 parts

Commit message: Dodano zabezpieczenia
Changed lines of the file:
@@
 $Descr A4 11693 8268
 encoding utf-8
-Sheet 1 6
+Sheet 1 5
 Title ""
 Date ""
@@
 $EndSheet
 $Sheet
-S 7450 1050 1650 1750
-U 67A7C74A
-F0 "Power" 50
-F1 "Power.sch" 50
-$EndSheet
-$Sheet
 S 2750 3200 1850 1250
 U 67A7C799
@@
 $EndSheet
 $Sheet
-S 5300 3250 1650 1400
-U 67A80A69
-F0 "CurrentSense" 50
-F1 "Cs.sch" 50
+S 5050 3100 2200 1400
+U 67AFAEB3
+F0 "Power And motor protection" 50
+F1 "Power and motor protection.sch" 50
 $EndSheet
 $EndSCHEMATC
