File: Hardware/C10W1B1V1.0/Kicad/Cs.sch (KiCad schematic (older format))
At the start: 1 part, among them IC2 TSC101AILT

Commit message: Dodano zabezpieczenia
Parts:
- removed IC2: TSC101AILT, Footprints:SOT95P280X145-5N, symbol TSC101AILT:TSC101AILT
Changed lines of the file:
@@
 $Descr A4 11693 8268
 encoding utf-8
-Sheet 6 6
+Sheet 6 7
 Title ""
 Date ""
@@
 Comment4 ""
 $EndDescr
-$Comp
-L TSC101AILT:TSC101AILT IC2
-U 1 1 67A80F7A
-P 4600 2400
-F 0 "IC2" H 5100 2665 50  0000 C CNN
-F 1 "TSC101AILT" H 5100 2574 50  0000 C CNN
-F 2 "Footprints:SOT95P280X145-5N" H 5450 2500 50  0001 L CNN
-F 3 "http://www.st.com/st-web-ui/static/active/en/resource/technical/document/datasheet/CD00153725.pdf" H 5450 2400 50  0001 L CNN
-F 4 "TSC101AILT, Current Sensing Amplifier Single 5-Pin SOT-23" H 5450 2300 50  0001 L CNN "Description"
-F 5 "1.45" H 5450 2200 50  0001 L CNN "Height"
-F 6 "STMicroelectronics" H 5450 2100 50  0001 L CNN "Manufacturer_Name"
-F 7 "TSC101AILT" H 5450 2000 50  0001 L CNN "Manufacturer_Part_Number"
-F 8 "511-TSC101AILT" H 5450 1900 50  0001 L CNN "Mouser Part Number"
-F 9 "https://www.mouser.co.uk/ProductDetail/STMicroelectronics/TSC101AILT?qs=lcekmG%2FW9swbeAXhKLEWhg%3D%3D" H 5450 1800 50  0001 L CNN "Mouser Price/Stock"
-F 10 "TSC101AILT" H 5450 1700 50  0001 L CNN "Arrow Part Number"
-F 11 "https://www.arrow.com/en/products/tsc101ailt/stmicroelectronics" H 5450 1600 50  0001 L CNN "Arrow Price/Stock"
-	1    4600 2400
-	1    0    0    -1
-$EndComp
 $EndSCHEMATC
