File: Hardware/C10W1B1V1.0/Kicad/H-Bridge.sch (KiCad schematic (older format))
At the start: 22 parts, among them Q1 STL300N4LF8, Q2 SI7155DP-T1-GE3, Q3 STL300N4LF8, Q4 SI7155DP-T1-GE3, Q5 SQ2362CES-T1_GE3, Q6 SQ2362CES-T1_GE3

Commit message: Dodano zabezpieczenia
Parts:
- R1, R12, R8, R9: value 10K/1%/0.063W -> 1K/1%/0.063W
Changed lines of the file:
@@
 $Descr A4 11693 8268
 encoding utf-8
-Sheet 3 6
+Sheet 3 5
 Title ""
 Date ""
@@
 P 2650 2550
 F 0 "R1" V 2650 2500 50  0000 L CNN
-F 1 "10K/1%/0.063W" V 2550 2250 50  0000 L CNN
+F 1 "1K/1%/0.063W" V 2550 2250 50  0000 L CNN
 F 2 "Resistor_SMD:R_0402_1005Metric" V 2580 2550 50  0001 C CNN
 F 3 "~" H 2650 2550 50  0001 C CNN
@@
 P 8750 2550
 F 0 "R8" V 8750 2500 50  0000 L CNN
-F 1 "10K/1%/0.063W" V 8650 2250 50  0000 L CNN
+F 1 "1K/1%/0.063W" V 8650 2250 50  0000 L CNN
 F 2 "Resistor_SMD:R_0402_1005Metric" V 8680 2550 50  0001 C CNN
 F 3 "~" H 8750 2550 50  0001 C CNN
@@
 P 8750 3900
 F 0 "R12" V 8750 3850 50  0000 L CNN
-F 1 "10K/1%/0.063W" V 8650 3600 50  0000 L CNN
+F 1 "1K/1%/0.063W" V 8650 3600 50  0000 L CNN
 F 2 "Resistor_SMD:R_0402_1005Metric" V 8680 3900 50  0001 C CNN
 F 3 "~" H 8750 3900 50  0001 C CNN
@@
 P 2650 3900
 F 0 "R9" V 2650 3850 50  0000 L CNN
-F 1 "10K/1%/0.063W" V 2550 3600 50  0000 L CNN
+F 1 "1K/1%/0.063W" V 2550 3600 50  0000 L CNN
 F 2 "Resistor_SMD:R_0402_1005Metric" V 2580 3900 50  0001 C CNN
 F 3 "~" H 2650 3900 50  0001 C CNN
