File: Hardware/C10W1B1V1.0/Kicad/uC.sch (KiCad schematic (older format))
At the start: 1 part, among them IC1 STM32L412K8U6

Commit message: Dodano zabezpieczenia
Parts:
- removed IC1: STM32L412K8U6, QFN50P500X500X60-33N-D, symbol STM32L412K8U6:STM32L412K8U6
- added C31, C32, C33, C34, C35: 4u7/50V/X5R, Capacitor_SMD:C_0402_1005Metric, symbol Device:C
- added D7, D8, D?: BAT54S, Package_TO_SOT_SMD:SOT-23, symbol Diode:BAT54S
- added R27, R28, R?: 10K/1%/0.063W, Resistor_SMD:R_0402_1005Metric, symbol Device:R
- added R29, R31: 174K/1%/0.063W, Resistor_SMD:R_0402_1005Metric, symbol Device:R
- added R30, R32: 330K/1%/0.063W, Resistor_SMD:R_0402_1005Metric, symbol Device:R
- added R?: 100K/1%/0.063W, Resistor_SMD:R_0402_1005Metric, symbol Device:R
- added U11: STM32L431CCUx, Package_DFN_QFN:QFN-48-1EP_7x7mm_P0.5mm_EP5.6x5.6mm, symbol MCU_ST_STM32L4:STM32L431CCUx
Connections:
- new net: R27.1, U11.44 (PH3)
- new net: R28.2, U11.7 (NRST)
- new net +3V3: C31.1, C32.1, C33.1, C34.1, C35.1, D7.2, D8.2, D?.2, R28.1, U11.1 (VBAT), U11.24 (VDD), U11.36 (VDDUSB), U11.48 (VDD), U11.9 (VDDA)
- new net ADC_IN5: D7.3, R29.2, R30.1, U11.10 (PA0)
- new net ADC_IN8: D?.3, R?.1, R?.2, U11.13 (PA3)
- new net ADC_IN9: D8.3, R31.2, R32.1, U11.14 (PA4)
- new net COMP_OUT: U11.41 (PB5)
- new net DBG_RX: U11.38 (PA15)
- new net DBG_TX: U11.12 (PA2)
- new net ENCODER_IN1: U11.15 (PA5)
- new net ENCODER_IN2: U11.11 (PA1)
- new net FLASH_CS: U11.22 (PB11)
- new net FLASH_IO0: U11.19 (PB1)
- new net FLASH_IO1: U11.18 (PB0)
- new net FLASH_IO2: U11.17 (PA7)
- new net FLASH_IO3: U11.16 (PA6)
- new net FLASH_SCK: U11.21 (PB10)
- new net FLOP_OUT: U11.25 (PB12)
- new net FRAM_CS: U11.20 (PB2)
- new net FRAM_MISO: U11.27 (PB14)
- new net FRAM_MOSI: U11.28 (PB15)
- new net FRAM_SCK: U11.26 (PB13)
- new net GND: C31.2, C32.2, C33.2, C34.2, C35.2, D7.1, D8.1, D?.1, R27.2, R30.2, R32.2, R?.2, U11.23 (VSS), U11.35 (VSS), U11.47 (VSS), U11.49 (VSS), U11.8 (VSSA)
- new net H_L_L_uC: U11.31 (PA10)
- new net H_L_R_uC: U11.32 (PA11)
- new net H_T_L_uC: U11.29 (PA8)
- new net H_T_R_uC: U11.30 (PA9)
- new net MAIN_CURRENT_SENSE: R29.1
- new net RX: U11.43 (PB7)
- new net SHORT_RANGE_CURRENT_SENSE: R31.1
- new net SHORT_RANGE_CURRENT_SENSE_EN: U11.33 (PA12)
- new net STARTUP_ENABLE: U11.46 (PB9)
- new net SWCLK: U11.37 (PA14)
- new net SWDIO: U11.34 (PA13)
- new net TX: U11.42 (PB6)
- new net VCC: R?.1
- new net ~FLOP_RST: U11.45 (PB8)
- no-connect marks 2 -> 6
